File: pcbs/kerigokbd_v1/kerigokbd.kicad_sch (KiCad schematic)
At the start: 85 parts, among them J1 USB4520-03-0-A, J2 Conn_01x04, J3 Conn_01x03, J4 SJ-3501-SMT-TR, SW1 SW_Push, SW10 SW_Push, SW11 SW_Push, SW12 SW_Push, SW13 SW_Push, SW14 SW_Push, SW15 SW_Push, SW16 SW_Push, SW17 SW_Push, SW18 SW_Push, SW19 SW_Push, SW2 SW_Push, SW20 SW_Push, SW21 SW_Push, SW22 SW_Push, SW23 SW_Push, SW24 SW_Push, SW3 SW_Push, SW4 SW_Push, SW5 SW_Push, SW6 SW_Push, SW7 SW_Push, SW8 SW_Push, SW9 SW_Push, U1 TLV75533PDBVR, U2 RP2040, U3 W25Q16JVUXIQ, Y1 12MHz

Commit message: update pcb
Parts:
- added JP2: LED_EN, Jumper:SolderJumper-2_P1.3mm_Bridged_RoundedPad1.0x1.5mm, symbol Jumper:SolderJumper_2_Bridged
- JP1: symbol Jumper:Jumper_2_Small_Open -> Jumper:SolderJumper_2_Open; now left out of the parts list
Connections:
- net GND: now also JP2.1 (A); no longer LED1.3 (VSS), LED10.3 (VSS), LED11.3 (VSS), LED12.3 (VSS), LED13.3 (VSS), LED14.3 (VSS), LED15.3 (VSS), LED16.3 (VSS), LED17.3 (VSS), LED18.3 (VSS), LED19.3 (VSS), LED2.3 (VSS), LED20.3 (VSS), LED21.3 (VSS), LED22.3 (VSS), LED23.3 (VSS), LED24.3 (VSS), LED3.3 (VSS), LED4.3 (VSS), LED5.3 (VSS), LED6.3 (VSS), LED7.3 (VSS), LED8.3 (VSS), LED9.3 (VSS)
- new net LED_GND: JP2.2 (B), LED1.3 (VSS), LED10.3 (VSS), LED11.3 (VSS), LED12.3 (VSS), LED13.3 (VSS), LED14.3 (VSS), LED15.3 (VSS), LED16.3 (VSS), LED17.3 (VSS), LED18.3 (VSS), LED19.3 (VSS), LED2.3 (VSS), LED20.3 (VSS), LED21.3 (VSS), LED22.3 (VSS), LED23.3 (VSS), LED24.3 (VSS), LED3.3 (VSS), LED4.3 (VSS), LED5.3 (VSS), LED6.3 (VSS), LED7.3 (VSS), LED8.3 (VSS), LED9.3 (VSS)
Changed lines of the file:
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@@
 	)
 	(junction
+		(at 196.85 87.63)
+		(diameter 0)
+		(color 0 0 0 0)
+	)
+	(junction
 		(at 196.85 77.47)
 		(diameter 0)
@@
 	)
 	(junction
-		(at 281.94 95.25)
-		(diameter 0)
-		(color 0 0 0 0)
-	)
-	(junction
 		(at 76.2 97.79)
 		(diameter 0)
@@
 	)
 	(junction
+		(at 227.33 95.25)
+		(diameter 0)
+		(color 0 0 0 0)
+	)
+	(junction
 		(at 33.02 167.64)
 		(diameter 0)
@@
 	(wire
 		(pts
+			(xy 196.85 95.25) (xy 227.33 95.25)
+		)
+		(stroke
+			(width 0)
+			(type default)
+		)
+	)
+	(wire
+		(pts
 			(xy 281.94 41.91) (xy 281.94 59.69)
 		)
@@
 	(wire
 		(pts
+			(xy 196.85 87.63) (xy 196.85 95.25)
+		)
+		(stroke
+			(width 0)
+			(type default)
+		)
+	)
+	(wire
+		(pts
 			(xy 50.8 85.09) (xy 58.42 85.09)
 		)
@@
 	(wire
 		(pts
+			(xy 185.42 87.63) (xy 196.85 87.63)
+		)
+		(stroke
+			(width 0)
+			(type default)
+		)
+	)
+	(wire
+		(pts
 			(xy 63.5 39.37) (xy 66.04 39.37)
 		)
@@
 	(text "LDO"
 		(exclude_from_sim no)
-		(at 99.441 21.082 0)
+		(at 92.964 23.114 0)
 		(effects
 			(font
@@
 		)
 	)
+	(label "LED_GND"
+		(at 185.42 87.63 0)
+		(fields_autoplaced yes)
+		(effects
+			(font
+				(size 1.27 1.27)
+			)
+			(justify left bottom)
+		)
+	)
 	(label "QSPI_SD2"
 		(at 45.72 135.89 180)
@@
 	)
 	(label "SPLIT_HAND"
-		(at 153.67 124.46 90)
+		(at 153.67 123.19 90)
 		(fields_autoplaced yes)
 		(effects
@@
 	(symbol
 		(lib_id "power:GND")
-		(at 153.67 129.54 0)
+		(at 153.67 130.81 0)
 		(unit 1)
 		(exclude_from_sim no)
@@
 		(fields_autoplaced yes)
 		(property "Reference" "#PWR035"
-			(at 153.67 135.89 0)
+			(at 153.67 137.16 0)
 			(effects
 				(font
@@
 		)
 		(property "Value" "GND"
-			(at 153.67 133.985 0)
+			(at 153.67 135.255 0)
 			(effects
 				(font
@@
 		)
 		(property "Footprint" ""
-			(at 153.67 129.54 0)
+			(at 153.67 130.81 0)
 			(effects
 				(font
@@
 		)
 		(property "Datasheet" ""
-			(at 153.67 129.54 0)
+			(at 153.67 130.81 0)
 			(effects
 				(font
@@
 		)
 		(property "Description" ""
-			(at 153.67 129.54 0)
+			(at 153.67 130.81 0)
 			(effects
 				(font
@@
 	)
 	(symbol
+		(lib_id "Jumper:SolderJumper_2_Bridged")
+		(at 181.61 87.63 0)
+		(unit 1)
+		(exclude_from_sim yes)
+		(in_bom no)
+		(on_board yes)
+		(dnp no)
+		(property "Reference" "JP2"
+			(at 181.61 82.804 0)
+			(effects
+				(font
+					(size 1.27 1.27)
+				)
+			)
+		)
+		(property "Value" "LED_EN"
+			(at 181.61 85.09 0)
+			(effects
+				(font
+					(size 1.27 1.27)
+				)
+			)
+		)
+		(property "Footprint" "Jumper:SolderJumper-2_P1.3mm_Bridged_RoundedPad1.0x1.5mm"
+			(at 181.61 87.63 0)
+			(effects
+				(font
+					(size 1.27 1.27)
+				)
+				(hide yes)
+			)
+		)
+		(property "Datasheet" "~"
+			(at 181.61 87.63 0)
+			(effects
+				(font
+					(size 1.27 1.27)
+				)
+				(hide yes)
+			)
+		)
+		(property "Description" "Solder Jumper, 2-pole, closed/bridged"
+			(at 181.61 87.63 0)
+			(effects
+				(font
+					(size 1.27 1.27)
+				)
+				(hide yes)
+			)
+		)
+		(pin "2"
+		)
+		(pin "1"
+		)
+		(instances
+			(project ""
+				(path "/4cc5d416-57f5-4147-8183-e03ae6b1198a"
+					(reference "JP2")
+					(unit 1)
+				)
+			)
+		)
+	)
+	(symbol
 		(lib_id "Device:C_Small")
 		(at 80.01 87.63 0)
@@
 	)
 	(symbol
-		(lib_id "Jumper:Jumper_2_Small_Open")
+		(lib_id "Jumper:SolderJumper_2_Open")
 		(at 153.67 127 90)
 		(unit 1)
 		(exclude_from_sim yes)
-		(in_bom yes)
+		(in_bom no)
 		(on_board yes)
 		(dnp no)
 		(fields_autoplaced yes)
 		(property "Reference" "JP1"
-			(at 154.94 125.7299 90)
+			(at 156.21 125.7299 90)
 			(effects
 				(font
@@
 		)
 		(property "Value" "Split Right"
-			(at 154.94 128.2699 90)
+			(at 156.21 128.2699 90)
 			(effects
 				(font
@@
 			)
 		)
-		(property "Description" "Jumper, 2-pole, small symbol, open"
+		(property "Description" "Solder Jumper, 2-pole, open"
 			(at 153.67 127 0)
 			(effects
@@
 	)
 	(symbol
+		(lib_id "power:PWR_FLAG")
+		(at 196.85 87.63 0)
+		(unit 1)
+		(exclude_from_sim no)
+		(in_bom yes)
+		(on_board yes)
+		(dnp no)
+		(property "Reference" "#FLG04"
+			(at 196.85 85.725 0)
+			(effects
+				(font
+					(size 1.27 1.27)
+				)
+				(hide yes)
+			)
+		)
+		(property "Value" "PWR_FLAG"
+			(at 196.85 83.82 0)
+			(effects
+				(font
+					(size 1.27 1.27)
+				)
+			)
+		)
+		(property "Footprint" ""
+			(at 196.85 87.63 0)
+			(effects
+				(font
+					(size 1.27 1.27)
+				)
+				(hide yes)
+			)
+		)
+		(property "Datasheet" ""
+			(at 196.85 87.63 0)
+			(effects
+				(font
+					(size 1.27 1.27)
+				)
+				(hide yes)
+			)
+		)
+		(property "Description" ""
+			(at 196.85 87.63 0)
+			(effects
+				(font
+					(size 1.27 1.27)
+				)
+				(hide yes)
+			)
+		)
+		(pin "1"
+		)
+		(instances
+			(project "kerigokbd"
+				(path "/4cc5d416-57f5-4147-8183-e03ae6b1198a"
+					(reference "#FLG04")
+					(unit 1)
+				)
+			)
+		)
+	)
+	(symbol
 		(lib_id "power:GND")
 		(at 50.8 34.29 90)
@@
 	(symbol
 		(lib_id "power:GND")
-		(at 281.94 95.25 0)
+		(at 177.8 87.63 0)
 		(unit 1)
 		(exclude_from_sim no)
@@
 		(dnp no)
 		(property "Reference" "#PWR023"
-			(at 281.94 101.6 0)
+			(at 177.8 93.98 0)
 			(effects
 				(font
@@
 		)
 		(property "Value" "GND"
-			(at 282.067 99.6442 0)
+			(at 177.927 92.0242 0)
 			(effects
 				(font
@@
 		)
 		(property "Footprint" ""
-			(at 281.94 95.25 0)
+			(at 177.8 87.63 0)
 			(effects
 				(font
@@
 		)
 		(property "Datasheet" ""
-			(at 281.94 95.25 0)
+			(at 177.8 87.63 0)
 			(effects
 				(font
@@
 		)
 		(property "Description" ""
-			(at 281.94 95.25 0)
+			(at 177.8 87.63 0)
 			(effects
 				(font

Commit message: update pcb
Parts:
- LED13, LED20: footprint kbd_local:YS-SK6812MINI-E -> kbd_local:YS-SK6812MINI-E-dual
Changed lines of the file:
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@@
 			)
 		)
-		(property "Footprint" "kbd_local:YS-SK6812MINI-E"
+		(property "Footprint" "kbd_local:YS-SK6812MINI-E-dual"
 			(at 275.59 76.2 0)
 			(effects
@@
 			)
 		)
-		(property "Footprint" "kbd_local:YS-SK6812MINI-E"
+		(property "Footprint" "kbd_local:YS-SK6812MINI-E-dual"
 			(at 275.59 58.42 0)
 			(effects
