File: keyboards/kerigokbd/pcb/kerigokbd.kicad_pcb (KiCad board)
At the start: 2 copper layers, 139.5 x 92 mm, 82 parts, among them J1 USB4520-03-0-A, J2 SDA SCL 5V GND, J3 SWC SWD GND, J4 SJ-3501-SMT-TR, SW1 SW_Push, SW10 SW_Push, SW11 SW_Push, SW12 SW_Push, SW13 SW_Push, SW14 SW_Push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

Commit message: mv pcb
Parts:
- J1, J4: moved to B.Cu
- turned J1 to 0 degrees
- turned J4 to 90 degrees
