File: hardware/kerigokbd_v1/pcb/kerigokbd.kicad_sch (KiCad schematic)
At the start: 86 parts, among them J1 USB4520-03-0-A, J2 Conn_01x04, J3 Conn_01x03, J4 SJ-3501-SMT-TR, SW1 SW_Push, SW10 SW_Push, SW11 SW_Push, SW12 SW_Push, SW13 SW_Push, SW14 SW_Push, SW15 SW_Push, SW16 SW_Push, SW17 SW_Push, SW18 SW_Push, SW19 SW_Push, SW2 SW_Push, SW20 SW_Push, SW21 SW_Push, SW22 SW_Push, SW23 SW_Push, SW24 SW_Push, SW3 SW_Push, SW4 SW_Push, SW5 SW_Push, SW6 SW_Push, SW7 SW_Push, SW8 SW_Push, SW9 SW_Push, U1 TLV75533PDBVR, U2 RP2040, U3 W25Q16JVUXIQ, Y1 12MHz

Commit message: update kicad 3d path
Parts:
- J2: value Conn_01x04 -> I2C
- J3: value Conn_01x03 -> SWD
Changed lines of the file:
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@@
 			)
 		)
-		(property "Value" "Conn_01x04"
+		(property "Value" "I2C"
 			(at 127 61.722 0)
 			(effects
@@
 			)
 		)
-		(property "Value" "Conn_01x03"
+		(property "Value" "SWD"
 			(at 147.32 61.976 0)
 			(effects

Commit message: update sketch
Connections:
- net TX renamed SERIAL
Other:
- note added: "Flash Memory"
- note added: "Key Switches"
- note added: "Power"
- note added: "boot"
- note removed: "DEBUG"
- note removed: "Flash memory"
- note removed: "I2C"
- note removed: "Key switches"
- note removed: "POWER"
- note removed: "boot switch"
Changed lines of the file:
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@@
 		)
 	)
-	(text "Key switches"
+	(text "Key Switches"
 		(exclude_from_sim no)
 		(at 181.61 107.442 0)
@@
 	(text "Extention"
 		(exclude_from_sim no)
-		(at 123.444 51.816 0)
+		(at 123.444 57.404 0)
 		(effects
 			(font
@@
 		)
 	)
-	(text "POWER\n"
+	(text "Power"
 		(exclude_from_sim no)
 		(at 20.701 20.066 0)
@@
 		)
 	)
-	(text "I2C"
+	(text "boot"
 		(exclude_from_sim no)
-		(at 124.206 57.404 0)
-		(effects
-			(font
-				(size 1.27 1.27)
-			)
-			(justify left bottom)
-		)
-	)
-	(text "boot switch"
-		(exclude_from_sim no)
-		(at 128.016 175.768 0)
+		(at 125.222 175.514 0)
 		(effects
 			(font
@@
 	(text "TRS"
 		(exclude_from_sim no)
-		(at 123.825 108.331 0)
+		(at 119.888 107.95 0)
 		(effects
 			(font
@@
 		)
 	)
-	(text "Flash memory"
+	(text "Flash Memory"
 		(exclude_from_sim no)
-		(at 118.364 147.828 0)
+		(at 121.666 147.32 0)
 		(effects
 			(font
@@
 		)
 	)
-	(text "DEBUG"
-		(exclude_from_sim no)
-		(at 143.129 57.404 0)
-		(effects
-			(font
-				(size 1.27 1.27)
-			)
-			(justify left bottom)
-		)
-	)
 	(label "KEY2"
 		(at 96.52 113.03 0)
@@
 		)
 	)
-	(label "TX"
+	(label "SERIAL"
 		(at 135.89 121.92 0)
 		(fields_autoplaced yes)
@@
 		)
 	)
-	(label "TX"
+	(label "SERIAL"
 		(at 96.52 107.95 0)
 		(fields_autoplaced yes)
@@
 	(symbol
 		(lib_id "power:GND")
-		(at 87.63 57.15 0)
+		(at 83.82 63.5 0)
 		(unit 1)
 		(exclude_from_sim no)
@@
 		(dnp no)
 		(property "Reference" "#PWR013"
-			(at 87.63 63.5 0)
+			(at 83.82 69.85 0)
 			(effects
 				(font
@@
 		)
 		(property "Value" "GND"
-			(at 87.63 60.96 0)
+			(at 83.82 67.31 0)
 			(effects
 				(font
@@
 		)
 		(property "Footprint" ""
-			(at 87.63 57.15 0)
+			(at 83.82 63.5 0)
 			(effects
 				(font
@@
 		)
 		(property "Datasheet" ""
-			(at 87.63 57.15 0)
+			(at 83.82 63.5 0)
 			(effects
 				(font
@@
 		)
 		(property "Description" ""
-			(at 87.63 57.15 0)
+			(at 83.82 63.5 0)
 			(effects
 				(font
@@
 	(symbol
 		(lib_id "power:+5V")
-		(at 77.47 57.15 0)
+		(at 73.66 63.5 0)
 		(unit 1)
 		(exclude_from_sim no)
@@
 		(dnp no)
 		(property "Reference" "#PWR012"
-			(at 77.47 60.96 0)
+			(at 73.66 67.31 0)
 			(effects
 				(font
@@
 		)
 		(property "Value" "+5V"
-			(at 77.47 52.832 0)
+			(at 73.66 59.182 0)
 			(effects
 				(font
@@
 		)
 		(property "Footprint" ""
-			(at 77.47 57.15 0)
+			(at 73.66 63.5 0)
 			(effects
 				(font
@@
 		)
 		(property "Datasheet" ""
-			(at 77.47 57.15 0)
+			(at 73.66 63.5 0)
 			(effects
 				(font
@@
 		)
 		(property "Description" ""
-			(at 77.47 57.15 0)
+			(at 73.66 63.5 0)
 			(effects
 				(font
@@
 	(symbol
 		(lib_id "power:VBUS")
-		(at 67.31 57.15 0)
+		(at 63.5 63.5 0)
 		(unit 1)
 		(exclude_from_sim no)
@@
 		(fields_autoplaced yes)
 		(property "Reference" "#PWR011"
-			(at 67.31 60.96 0)
+			(at 63.5 67.31 0)
 			(effects
 				(font
@@
 		)
 		(property "Value" "VBUS"
-			(at 67.31 52.07 0)
+			(at 63.5 58.42 0)
 			(effects
 				(font
@@
 		)
 		(property "Footprint" ""
-			(at 67.31 57.15 0)
+			(at 63.5 63.5 0)
 			(effects
 				(font
@@
 		)
 		(property "Datasheet" ""
-			(at 67.31 57.15 0)
+			(at 63.5 63.5 0)
 			(effects
 				(font
@@
 		)
 		(property "Description" ""
-			(at 67.31 57.15 0)
+			(at 63.5 63.5 0)
 			(effects
 				(font
@@
 	(symbol
 		(lib_id "power:PWR_FLAG")
-		(at 67.31 57.15 180)
+		(at 63.5 63.5 180)
 		(unit 1)
 		(exclude_from_sim no)
@@
 		(dnp no)
 		(property "Reference" "#FLG01"
-			(at 67.31 59.055 0)
+			(at 63.5 65.405 0)
 			(effects
 				(font
@@
 		)
 		(property "Value" "PWR_FLAG"
-			(at 67.31 60.96 0)
+			(at 63.5 67.31 0)
 			(effects
 				(font
@@
 		)
 		(property "Footprint" ""
-			(at 67.31 57.15 0)
+			(at 63.5 63.5 0)
 			(effects
 				(font
@@
 		)
 		(property "Datasheet" ""
-			(at 67.31 57.15 0)
+			(at 63.5 63.5 0)
 			(effects
 				(font
@@
 		)
 		(property "Description" ""
-			(at 67.31 57.15 0)
+			(at 63.5 63.5 0)
 			(effects
 				(font
@@
 	(symbol
 		(lib_id "power:PWR_FLAG")
-		(at 87.63 57.15 0)
+		(at 83.82 63.5 0)
 		(unit 1)
 		(exclude_from_sim no)
@@
 		(dnp no)
 		(property "Reference" "#FLG03"
-			(at 87.63 55.245 0)
+			(at 83.82 61.595 0)
 			(effects
 				(font
@@
 		)
 		(property "Value" "PWR_FLAG"
-			(at 87.63 53.34 0)
+			(at 83.82 59.69 0)
 			(effects
 				(font
@@
 		)
 		(property "Footprint" ""
-			(at 87.63 57.15 0)
+			(at 83.82 63.5 0)
 			(effects
 				(font
@@
 		)
 		(property "Datasheet" ""
-			(at 87.63 57.15 0)
+			(at 83.82 63.5 0)
 			(effects
 				(font
@@
 		)
 		(property "Description" ""
-			(at 87.63 57.15 0)
+			(at 83.82 63.5 0)
 			(effects
 				(font
@@
 	(symbol
 		(lib_id "power:PWR_FLAG")
-		(at 77.47 57.15 180)
+		(at 73.66 63.5 180)
 		(unit 1)
 		(exclude_from_sim no)
@@
 		(dnp no)
 		(property "Reference" "#FLG02"
-			(at 77.47 59.055 0)
+			(at 73.66 65.405 0)
 			(effects
 				(font
@@
 		)
 		(property "Value" "PWR_FLAG"
-			(at 77.47 60.96 0)
+			(at 73.66 67.31 0)
 			(effects
 				(font
@@
 		)
 		(property "Footprint" ""
-			(at 77.47 57.15 0)
+			(at 73.66 63.5 0)
 			(effects
 				(font
@@
 		)
 		(property "Datasheet" ""
-			(at 77.47 57.15 0)
+			(at 73.66 63.5 0)
 			(effects
 				(font
@@
 		)
 		(property "Description" ""
-			(at 77.47 57.15 0)
+			(at 73.66 63.5 0)
 			(effects
 				(font

Commit message: update docs and images
Other:
- title: KERIgoKBD -> KERIgoKBD v1
Changed lines of the file:
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@@
 	(paper "A4")
 	(title_block
-		(title "KERIgoKBD")
-		(date "2024-12-27")
+		(title "KERIgoKBD v1")
+		(date "2024-12-29")
 		(rev "1.0.0")
 		(company "KERI's Lab")

Commit message: update sketch
Parts:
- added ZD2: NSR0520V2T5G, Diode_SMD:D_SOD-523, symbol Diode:ESD5Zxx
- SW1, SW10, SW11, SW12, SW13, SW14, SW15, SW16, SW17, SW18, SW19, SW2, SW20, SW21, SW22, SW23, SW24, SW3, SW4, SW5, SW6, SW7, SW8, SW9: value SW_Push -> Key_SW
Connections:
- net +3V3: now also J2.3 (Pin_3), ZD2.1 (K)
- net +5V: no longer J2.3 (Pin_3)
- net GND: now also J3.2 (Pin_2); no longer J3.3 (Pin_3)
- net LED: now also U2.2 (GPIO0); no longer U2.37 (GPIO25)
- net SCL: now also U2.39 (GPIO27_ADC1); no longer U2.40 (GPIO28_ADC2)
- net SDA: now also U2.38 (GPIO26_ADC0); no longer U2.41 (GPIO29_ADC3)
- net SERIAL: now also U2.41 (GPIO29_ADC3), ZD2.2 (A); no longer U2.2 (GPIO0)
- net SPLIT_HAND: now also U2.37 (GPIO25); no longer U2.39 (GPIO27_ADC1)
- net SWD: now also J3.3 (Pin_3); no longer J3.2 (Pin_2)
- net USB_VBUS_PIN: now also U2.40 (GPIO28_ADC2); no longer U2.38 (GPIO26_ADC0)
- no-connect marks 3 -> 4
Other:
- note added: "Key Switch"
- note added: "LED"
- note removed: "Key Switches"
- note removed: "LDO"
- note removed: "LEDs"
- note removed: "VBUS ESD"
- note removed: "close to pin 44"
- note removed: "close to pin 45"
- moved on the sheet: C1, C2, J2, J3, J4, JP1, U1

Commit message: update pcb
Parts:
- renumbered JP2 to JP1, JP1 to JP2
Connections:
- net +3V3: no longer ZD2.1 (K)
- net GND: now also ZD2.2 (A)
- net SERIAL: now also ZD2.1 (K); no longer ZD2.2 (A)
Other:
- note added: "reset"
- moved on the sheet: C1, C2, J1, J2, J3, J4, JP2, R1, R2, R3, R4, U1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

Commit message: update sketch
Other:
- title: KERIgoKBD v1 -> KERIgoKBD v1.1

Commit message: update sketch
Parts:
- ZD2: value NSR0520V2T5G -> BZT52C3V3LP-7
Changed lines of the file:
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@@
 			)
 		)
-		(property "Value" "NSR0520V2T5G"
+		(property "Value" "BZT52C3V3LP-7"
 			(at 160.274 117.348 0)
 			(effects

Commit message: update PCB v2026.02.22a
Parts:
- removed JP1: LED_EN, Jumper:SolderJumper-2_P1.3mm_Bridged_RoundedPad1.0x1.5mm, symbol Jumper:SolderJumper_2_Bridged
- removed ZD2: BZT52C3V3LP-7, Diode_SMD:D_SOD-523, symbol Diode:ESD5Zxx
Connections:
- net LED_GND is gone; now on net GND: LED1.3 (VSS), LED10.3 (VSS), LED11.3 (VSS), LED12.3 (VSS), LED13.3 (VSS), LED14.3 (VSS), LED15.3 (VSS), LED16.3 (VSS), LED17.3 (VSS), LED18.3 (VSS), LED19.3 (VSS), LED2.3 (VSS), LED20.3 (VSS), LED21.3 (VSS), LED22.3 (VSS), LED23.3 (VSS), LED24.3 (VSS), LED3.3 (VSS), LED4.3 (VSS), LED5.3 (VSS), LED6.3 (VSS), LED7.3 (VSS), LED8.3 (VSS), LED9.3 (VSS)
- net +5V: now also J4.S; no longer J4.T
- net D+: no longer J1.B6 (D+)
- net D-: no longer J1.B7 (D-)
- net GND: now also J4.R; no longer J4.S
- net SERIAL: now also J4.T; no longer J4.R
- no-connect marks 4 -> 6
