File: hardware/kerigokbd_v1/pcb/kerigokbd.kicad_sch (KiCad schematic)
At the start: 85 parts, among them J1 USB4520-03-0-A, J2 I2C, J3 SWD, J4 SJ-3501-SMT-TR, SW1 Key_SW, SW10 Key_SW, SW11 Key_SW, SW12 Key_SW, SW13 Key_SW, SW14 Key_SW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

Commit message: update svg and pdf
Other:
- title: KERIgoKBD v1.1 -> KERIgoKBD v1.2
Changed lines of the file:
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@@
 	(paper "A4")
 	(title_block
-		(title "KERIgoKBD v1.1")
-		(date "2025-02-08")
-		(rev "1.1.0")
+		(title "KERIgoKBD v1.2")
+		(date "2026-02-22")
+		(rev "1.2.0")
 		(company "KERI's Lab")
 	)
